Commit message: Add hokuyo lidar

File: simulator_ws/src/tb_gazebo_description/robots/kobuki_hexagons_kinect.urdf.xacro (robot description, xacro)
@@ -10,6 +10,10 @@
   <xacro:include filename="$(find tb_gazebo_description)/urdf/stacks/hexagons.urdf.xacro"/>
   <xacro:include filename="$(find tb_gazebo_description)/urdf/sensors/kinect.urdf.xacro"/>
+  <xacro:include filename="$(find tb_gazebo_description)/urdf/sensors/hokuyo_utm30lx.urdf.xacro"/>
   <kobuki/>
   <stack_hexagons parent="base_link"/>
   <sensor_kinect  parent="base_link"/>
+  <hokuyo_utm30lx_gpu name="hokuyo_laser" parent="base_link" ros_topic="/hokuyo_laser" update_rate="30" ray_count="720" min_angle="0" max_angle="360">
+    <origin xyz="0 0 +0.10" rpy="0 0 0" />
+  </hokuyo_utm30lx_gpu>
 </robot>
